File: hw/rascsi_2p7/Connectors.kicad_sch (KiCad schematic)
At the start: 3 parts

Commit message: as-ordered v2.7a
Parts:
- J20: LCSC (none) -> DNP
Changed lines of the file:
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@@
       (effects (font (size 1.27 1.27)) (justify left) hide)
+    )
+    (property "LCSC" "DNP" (id 10) (at 157.48 36.83 0)
+      (effects (font (size 1.27 1.27)) hide)
     )
     (pin "1")
