File: hw/rascsi_2p7/rascsi_2p7.kicad_pcb (KiCad board)
At the start: 2 copper layers, 65 x 56 mm, 96 parts, among them IC1 SN74LVT245BPWR, IC2 SN74LVT245BPWR, IC3 SN74LVT245BPWR, IC4 SN74LVT245BPWR, J1 Raspberry_Pi_2_3, J2 DNP, J20 171826-4, J3 Conn_02x25_Odd_Even, J4 I2C Pinout, J5 DNP, J6 CONNFLY DB-25, J8 USB_B_Micro, J9 Conn_02x25_Odd_Even, X1 Mac, X2 Dogcow, X3 Mac, X4 Dogcow, X5 Dogcow, X6 Dogcow, X7 Pi, X8 Pi, X9 CE Logo

Commit message: as-ordered v2.7a
Parts:
- moved FUSE1 6.76 mm to (204.4, 73.7)
- moved D5 2.03 mm to (204.4, 68.4), turned to 90 degrees
- moved X5 0.52 mm to (212.6, 57.8)
- moved X6 0.40 mm to (199.6, 57.8)
- moved X4 0.14 mm to (225.6, 57.8)
- moved X2 0.11 mm to (186.7, 57.8)
Routing:
- net TERMPOW: track 51.7 -> 44.6 mm
- net C-RST: vias 5 -> 4
Other:
- board text added: "Version 2.7a"
- board text removed: "Version 2.6c"
