File: hw/rascsi_2p7/rascsi_2p7.kicad_sch (KiCad schematic)
At the start: 89 parts

Commit message: as-ordered v2.7a
Parts:
- R23, R24, R25, R26, R27, R28, R29, R30, R31, R32, R33, R34, R35, R36, R37, R38, R39, R40: LCSC C17557 -> C163392; Manufacturer_Name UNI-ROYAL(Uniroyal Elec) -> YAGEO; Manufacturer_Part_Number 0805W8F2200T5E -> RC0805JR-7W220RL
- R41, R42, R43, R44, R45, R46, R47, R48, R49, R50, R51, R52, R53, R54, R55, R56, R57, R58: LCSC C17630 -> C365291; Manufacturer_Name UNI-ROYAL(Uniroyal Elec) -> Resistor.Today; Manufacturer_Part_Number 0805W8F3300T5E -> HPCR0805F330RK9
Other:
- note added: "2.7"
- note removed: "2.6"
