File: hw/daisy_chain_board/daisy_chain_board.kicad_sch (KiCad schematic)
At the start: 9 parts

Commit message: delete extraneous files
Parts:
- H5: value (none) -> Hole4; footprint (none) -> MountingHole:MountingHole_2.7mm
- H6: value (none) -> Hole6; footprint (none) -> MountingHole:MountingHole_2.7mm
- J7: value (none) -> Conn_02x25_Odd_Even; footprint (none) -> Connector_PinHeader_2.54mm:PinHeader_2x25_P2.54mm_Vertical
- J8: value (none) -> CONFLY DB25; footprint (none) -> L717SDB25PA4CH4F
- X1: value (none) -> Mac; footprint (none) -> SamacSys_Parts:mac_happy_small
- X2: value (none) -> Dogcow; footprint (none) -> SamacSys_Parts:dogcow
- X3: value (none) -> Mac2; footprint (none) -> SamacSys_Parts:mac_happy_small
- X4: value (none) -> Raspberry Pi; footprint (none) -> SamacSys_Parts:pi_logo
- X7: value (none) -> Pi; footprint (none) -> SamacSys_Parts:pi_logo
Other:
- note added: "3-Sept-2022"
- note added: "v2"
- note removed: "19-Aug-2020"
- note removed: "2.2"
Changed lines of the file:
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@@
     (stroke (width 0) (type default) (color 0 0 0 0))
   )
-  (text "2.2" (at 251.46 200.406 0)
+  (text "v2" (at 251.46 200.406 0)
     (effects (font (size 2.0066 2.0066) (thickness 0.4013) bold) (justify left bottom))
   )
@@
     (effects (font (size 1.27 1.27)) (justify left bottom))
   )
-  (text "19-Aug-2020" (at 189.23 199.898 0)
+  (text "3-Sept-2022" (at 189.23 199.898 0)
     (effects (font (size 1.4986 1.4986) (thickness 0.2997) bold) (justify left bottom))
   )
@@
     (in_bom yes) (on_board yes)
     (property "Reference" "J7" (id 0) (at 126.365 52.07 0))
-    (property "Value" "" (id 1) (at 124.0536 52.07 0))
-    (property "Footprint" "" (id 2) (at 90.17 53.34 0)
+    (property "Value" "Conn_02x25_Odd_Even" (id 1) (at 124.0536 52.07 0))
+    (property "Footprint" "Connector_PinHeader_2.54mm:PinHeader_2x25_P2.54mm_Vertical" (id 2) (at 90.17 53.34 0)
       (effects (font (size 1.27 1.27)) hide)
     )
@@
       (effects (font (size 1.27 1.27)) (justify left))
     )
-    (property "Value" "" (id 1) (at 64.77 135.6868 0)
-      (effects (font (size 1.27 1.27)) (justify left))
-    )
-    (property "Footprint" "" (id 2) (at 62.23 134.62 0)
+    (property "Value" "Hole4" (id 1) (at 64.77 135.6868 0)
+      (effects (font (size 1.27 1.27)) (justify left))
+    )
+    (property "Footprint" "MountingHole:MountingHole_2.7mm" (id 2) (at 62.23 134.62 0)
       (effects (font (size 1.27 1.27)) hide)
     )
@@
       (effects (font (size 1.27 1.27)) (justify left))
     )
-    (property "Value" "" (id 1) (at 74.93 135.6868 0)
-      (effects (font (size 1.27 1.27)) (justify left))
-    )
-    (property "Footprint" "" (id 2) (at 72.39 134.62 0)
+    (property "Value" "Hole6" (id 1) (at 74.93 135.6868 0)
+      (effects (font (size 1.27 1.27)) (justify left))
+    )
+    (property "Footprint" "MountingHole:MountingHole_2.7mm" (id 2) (at 72.39 134.62 0)
       (effects (font (size 1.27 1.27)) hide)
     )
@@
       (effects (font (size 1.27 1.27)) (justify left))
     )
-    (property "Value" "" (id 1) (at 58.42 152.4 0)
-      (effects (font (size 1.27 1.27)) (justify left))
-    )
-    (property "Footprint" "" (id 2) (at 57.15 154.94 0)
+    (property "Value" "Mac" (id 1) (at 58.42 152.4 0)
+      (effects (font (size 1.27 1.27)) (justify left))
+    )
+    (property "Footprint" "SamacSys_Parts:mac_happy_small" (id 2) (at 57.15 154.94 0)
       (effects (font (size 1.27 1.27)) hide)
     )
@@
       (effects (font (size 1.27 1.27)) (justify left))
     )
-    (property "Value" "" (id 1) (at 58.42 154.94 0)
-      (effects (font (size 1.27 1.27)) (justify left))
-    )
-    (property "Footprint" "" (id 2) (at 57.15 157.48 0)
+    (property "Value" "Dogcow" (id 1) (at 58.42 154.94 0)
+      (effects (font (size 1.27 1.27)) (justify left))
+    )
+    (property "Footprint" "SamacSys_Parts:dogcow" (id 2) (at 57.15 157.48 0)
       (effects (font (size 1.27 1.27)) hide)
     )
@@
       (effects (font (size 1.27 1.27)) (justify left))
     )
-    (property "Value" "" (id 1) (at 58.42 157.48 0)
-      (effects (font (size 1.27 1.27)) (justify left))
-    )
-    (property "Footprint" "" (id 2) (at 57.15 160.02 0)
+    (property "Value" "Mac2" (id 1) (at 58.42 157.48 0)
+      (effects (font (size 1.27 1.27)) (justify left))
+    )
+    (property "Footprint" "SamacSys_Parts:mac_happy_small" (id 2) (at 57.15 160.02 0)
       (effects (font (size 1.27 1.27)) hide)
     )
@@
       (effects (font (size 1.27 1.27)) (justify right))
     )
-    (property "Value" "" (id 1) (at 72.39 154.94 0)
-      (effects (font (size 1.27 1.27)) (justify right))
-    )
-    (property "Footprint" "" (id 2) (at 71.12 153.67 0)
+    (property "Value" "Raspberry Pi" (id 1) (at 72.39 154.94 0)
+      (effects (font (size 1.27 1.27)) (justify right))
+    )
+    (property "Footprint" "SamacSys_Parts:pi_logo" (id 2) (at 71.12 153.67 0)
       (effects (font (size 1.27 1.27)) hide)
     )
@@
       (effects (font (size 1.27 1.27)) (justify right))
     )
-    (property "Value" "" (id 1) (at 72.39 157.48 0)
-      (effects (font (size 1.27 1.27)) (justify right))
-    )
-    (property "Footprint" "" (id 2) (at 71.12 156.21 0)
+    (property "Value" "Pi" (id 1) (at 72.39 157.48 0)
+      (effects (font (size 1.27 1.27)) (justify right))
+    )
+    (property "Footprint" "SamacSys_Parts:pi_logo" (id 2) (at 71.12 156.21 0)
       (effects (font (size 1.27 1.27)) hide)
     )
@@
       (effects (font (size 1.27 1.27)) hide)
     )
-    (property "Value" "" (id 1) (at 120.777 65.3542 0))
+    (property "Value" "GND" (id 1) (at 120.777 65.3542 0))
     (property "Footprint" "" (id 2) (at 120.65 60.96 0)
       (effects (font (size 1.27 1.27)) hide)
@@
       (effects (font (size 1.27 1.27)) hide)
     )
-    (property "Value" "" (id 1) (at 76.9112 119.253 90)
+    (property "Value" "GND" (id 1) (at 76.9112 119.253 90)
       (effects (font (size 1.27 1.27)) (justify right))
     )
@@
       (effects (font (size 1.27 1.27)) hide)
     )
-    (property "Value" "" (id 1) (at 89.6112 81.153 90)
+    (property "Value" "GND" (id 1) (at 89.6112 81.153 90)
       (effects (font (size 1.27 1.27)) (justify right))
     )
@@
       (effects (font (size 1.27 1.27)) hide)
     )
-    (property "Value" "" (id 1) (at 89.6112 86.233 90)
+    (property "Value" "GND" (id 1) (at 89.6112 86.233 90)
       (effects (font (size 1.27 1.27)) (justify right))
     )
@@
       (effects (font (size 1.27 1.27)) hide)
     )
-    (property "Value" "" (id 1) (at 89.6112 91.313 90)
+    (property "Value" "GND" (id 1) (at 89.6112 91.313 90)
       (effects (font (size 1.27 1.27)) (justify right))
     )
@@
       (effects (font (size 1.27 1.27)) hide)
     )
-    (property "Value" "" (id 1) (at 57.7088 96.647 90)
+    (property "Value" "GND" (id 1) (at 57.7088 96.647 90)
       (effects (font (size 1.27 1.27)) (justify right))
     )
@@
       (effects (font (size 1.27 1.27)) hide)
     )
-    (property "Value" "" (id 1) (at 57.7088 101.727 90)
+    (property "Value" "GND" (id 1) (at 57.7088 101.727 90)
       (effects (font (size 1.27 1.27)) (justify right))
     )
@@
       (effects (font (size 1.27 1.27)) hide)
     )
-    (property "Value" "" (id 1) (at 89.6112 106.553 90)
+    (property "Value" "GND" (id 1) (at 89.6112 106.553 90)
       (effects (font (size 1.27 1.27)) (justify right))
     )
@@
       (effects (font (size 1.27 1.27)) hide)
     )
-    (property "Value" "" (id 1) (at 76.9112 73.533 90)
+    (property "Value" "GND" (id 1) (at 76.9112 73.533 90)
       (effects (font (size 1.27 1.27)) (justify right))
     )
@@
     (in_bom yes) (on_board yes)
     (property "Reference" "J8" (id 0) (at 73.66 69.0626 90))
-    (property "Value" "" (id 1) (at 73.66 71.374 90))
-    (property "Footprint" "" (id 2) (at 66.04 115.57 0)
+    (property "Value" "CONFLY DB25" (id 1) (at 73.66 71.374 90))
+    (property "Footprint" "L717SDB25PA4CH4F" (id 2) (at 66.04 115.57 0)
       (effects (font (size 1.27 1.27)) (justify left) hide)
     )

Commit message: re-add 3d shapes
Parts:
- removed X2: Dogcow, SamacSys_Parts:dogcow, symbol SamacSys_Parts:Logo
Changed lines of the file:
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@@
-    )
-  )
-  (symbol (lib_id "SamacSys_Parts:Logo") (at 57.15 157.48 0) (unit 1)
-    (in_bom yes) (on_board yes)
-    (property "Reference" "X2" (id 0) (at 53.34 154.94 0)
-      (effects (font (size 1.27 1.27)) (justify left))
-    )
-    (property "Value" "Dogcow" (id 1) (at 58.42 154.94 0)
-      (effects (font (size 1.27 1.27)) (justify left))
-    )
-    (property "Footprint" "SamacSys_Parts:dogcow" (id 2) (at 57.15 157.48 0)
-      (effects (font (size 1.27 1.27)) hide)
-    )
-    (property "Datasheet" "" (id 3) (at 57.15 157.48 0)
-      (effects (font (size 1.27 1.27)) hide)
     )
   )
@@
       (reference "X1") (unit 1) (value "Mac") (footprint "SamacSys_Parts:mac_happy_small")
     )
-    (path "/00000000-0000-0000-0000-00005efcd6ca"
-      (reference "X2") (unit 1) (value "Dogcow") (footprint "SamacSys_Parts:dogcow")
-    )
     (path "/00000000-0000-0000-0000-00005efcd8d2"

Commit message: As-ordered version
Other:
- note added: "8-Sept-2022"
- note removed: "3-Sept-2022"
Changed lines of the file:
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@@
     (effects (font (size 1.27 1.27)) (justify left bottom))
   )
-  (text "3-Sept-2022" (at 189.23 199.898 0)
+  (text "8-Sept-2022" (at 189.23 199.898 0)
     (effects (font (size 1.4986 1.4986) (thickness 0.2997) bold) (justify left bottom))
   )
@@
     (pin "MH2")
   )
+  (symbol (lib_id "power:PWR_FLAG") (at 109.22 110.49 0) (unit 1)
+    (in_bom yes) (on_board yes) (fields_autoplaced)
+    (property "Reference" "#FLG01" (id 0) (at 109.22 108.585 0)
+      (effects (font (size 1.27 1.27)) hide)
+    )
+    (property "Value" "PWR_FLAG" (id 1) (at 109.22 105.41 0))
+    (property "Footprint" "" (id 2) (at 109.22 110.49 0)
+      (effects (font (size 1.27 1.27)) hide)
+    )
+    (property "Datasheet" "~" (id 3) (at 109.22 110.49 0)
+      (effects (font (size 1.27 1.27)) hide)
+    )
+    (pin "1")
+  )
+  (symbol (lib_id "power:GND") (at 109.22 110.49 0) (unit 1)
+    (in_bom yes) (on_board yes)
+    (property "Reference" "#PWR01" (id 0) (at 109.22 116.84 0)
+      (effects (font (size 1.27 1.27)) hide)
+    )
+    (property "Value" "GND" (id 1) (at 109.347 114.8842 0))
+    (property "Footprint" "" (id 2) (at 109.22 110.49 0)
+      (effects (font (size 1.27 1.27)) hide)
+    )
+    (property "Datasheet" "" (id 3) (at 109.22 110.49 0)
+      (effects (font (size 1.27 1.27)) hide)
+    )
+    (pin "1")
+  )
   (sheet_instances
     (path "/" (page "1"))
   )
   (symbol_instances
+    (path "/4452e23f-c15a-4592-ad16-648fbd3cc29f"
+      (reference "#FLG01") (unit 1) (value "PWR_FLAG") (footprint "")
+    )
+    (path "/ea1ef6ed-ba99-4247-a667-818aeeda3964"
+      (reference "#PWR01") (unit 1) (value "GND") (footprint "")
+    )
     (path "/00000000-0000-0000-0000-00005f3086c0"
       (reference "#PWR015") (unit 1) (value "GND") (footprint "")
