File: hw/rascsi_2p6/Connectors.kicad_sch (KiCad schematic)
At the start: 3 parts, among them J20 171826-4, J3 Conn_02x25_Odd_Even, J9 Conn_02x25_Odd_Even

Commit message: as ordered
Parts:
- J20: LCSC (none) -> DNP
Changed lines of the file:
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@@
       (effects (font (size 1.27 1.27)) (justify left) hide)
+    )
+    (property "LCSC" "DNP" (id 10) (at 157.48 36.83 0)
+      (effects (font (size 1.27 1.27)) hide)
     )
     (pin "1")
