File: hw/rascsi_2p6/rascsi_2p6.kicad_pcb (KiCad board)
At the start: 2 copper layers, 65 x 56 mm, 98 parts, among them IC1 SN74F245DWR, IC2 SN74F245DWR, IC3 SN74F245DWR, IC4 SN74F245DWR, J1 Raspberry_Pi_2_3, J2 DNP, J20 171826-4, J3 Conn_02x25_Odd_Even, J4 I2C Pinout, J5 DNP, J6 CONNFLY DB-25, J8 USB_B_Micro, J9 Conn_02x25_Odd_Even, X1 Mac, X2 Dogcow, X3 Mac, X4 Dogcow, X5 Dogcow, X6 Dogcow, X7 Pi, X8 Pi

Commit message: as ordered
Parts:
- removed G***: LOGO, SamacSys_Parts:mac_happy_small
- removed REF**: CE-Logo_8.5x6mm_SilkScreen, Symbol:CE-Logo_8.5x6mm_SilkScreen
- removed REF**: KiCad-Logo_5mm_SilkScreen, Symbol:KiCad-Logo_5mm_SilkScreen
- IC1, IC2, IC3, IC4: value SN74F245DWR -> SN74LS641-1DW
- moved R19 5.97 mm to (196.5, 50.6)
- moved R20 5.97 mm to (197.7, 50.6)
- moved R21 5.97 mm to (199.0, 50.6)
- moved R22 5.97 mm to (200.3, 50.6)
Connections:
- IC1 pad 15: GND -> PI-DP
- IC1 pad 16: GND -> PI-D0
- IC1 pad 17: GND -> PI-D1
- IC1 pad 18: PI-DP -> PI-D2
- IC1 pad 2: C-DP -> C-D2
- IC1 pad 20: +3V3 -> +5V
- IC1 pad 3: GND -> C-D1
- IC1 pad 4: GND -> C-D0
- IC1 pad 5: GND -> C-DP
- IC2 pad 11: PI-D0 -> GND
- IC2 pad 12: PI-D1 -> GND
- IC2 pad 13: PI-D2 -> GND
- IC2 pad 20: +3V3 -> +5V
- IC2 pad 7: C-D2 -> GND
- IC2 pad 8: C-D1 -> GND
- IC2 pad 9: C-D0 -> GND
- IC3 pad 20: +3V3 -> +5V
- IC4 pad 20: +3V3 -> +5V
Routing:
- net GND: track 427.8 -> 484.2 mm, vias 28 -> 42
- net +5V: track 224.7 -> 244.3 mm, vias 6 -> 8
- net +3V3: track 158.3 -> 147.3 mm, vias 7 -> 6
- net PI-D2: track 48.2 -> 38.1 mm, vias 3 -> 1
- net PI-D1: track 26.0 -> 20.8 mm, vias 3 -> 2
- net PI-D0: track 16.8 -> 12.2 mm, vias 3 -> 1
- net PI-DP: track 10.9 -> 13.0 mm
- net PI-DTD: track 56.2 -> 54.2 mm
- net PI-MSG: track 19.8 -> 21.8 mm
- net PI-SEL: track 39.0 -> 37.8 mm
- net C-D0: track 95.6 -> 94.7 mm
- net PI_GPIO9: track 76.1 -> 75.4 mm
- net C-D7: track 60.5 -> 59.8 mm
- net PI-D6: track 47.6 -> 46.9 mm
- net PI-D3: track 40.0 -> 39.3 mm
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Other:
- board text added: "Reloaded Version 2.6d"
- board text removed: "Reloaded Version 2.6a"
