File: hw/rascsi_2p6/rascsi_2p6.kicad_sch (KiCad schematic)
At the start: 88 parts, among them IC1 SN74F245DWR, IC2 SN74F245DWR, IC3 SN74F245DWR, IC4 SN74F245DWR, J1 Raspberry_Pi_2_3, J2 DNP, J4 I2C Pinout, J5 DNP, J6 CONNFLY DB-25, X1 Mac, X2 Dogcow, X3 Mac, X4 Dogcow, X5 Dogcow, X6 Dogcow, X7 Pi, X8 Pi

Commit message: as ordered
Parts:
- IC1, IC2, IC3, IC4: value SN74F245DWR -> SN74LS641-1DW; LCSC C7165 -> C1548111; Manufacturer_Part_Number SN74F245DWR -> SN74LS641-1DW
- J6: value CONNFLY DB-25 -> (none); footprint SamacSys_Parts:L717SDB25PA4CH4F -> L717SDB25PA4CH4F; Height (none) -> 12.55; Manufacturer_Name CONNFLY Elec -> Amphenol; Manufacturer_Part_Number DS1037-25FNAKT74-0CC -> L717SDB25PA4CH4F; Mouser Part Number (none) -> 523-L717SDB25PA4CH4F; Mouser Price/Stock (none) -> https://www.mouser.com/Search/Refine.aspx?Keyword=523-L717S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
Connections:
- net +3V3: no longer IC1.20 (VCC), IC2.20 (VCC), IC3.20 (VCC), IC4.20 (VCC)
- net +5V: now also IC1.20 (VCC), IC2.20 (VCC), IC3.20 (VCC), IC4.20 (VCC)
- net C-D0: now also IC1.4 (A3); no longer IC2.9 (A8)
- net C-D1: now also IC1.3 (A2); no longer IC2.8 (A7)
- net C-D2: now also IC1.2 (A1); no longer IC2.7 (A6)
- net C-DP: now also IC1.5 (A4); no longer IC1.2 (A1)
- net GND: now also IC2.11 (B8), IC2.12 (B7), IC2.13 (B6), IC2.7 (A6), IC2.8 (A7), IC2.9 (A8); no longer IC1.15 (B4), IC1.16 (B3), IC1.17 (B2), IC1.3 (A2), IC1.4 (A3), IC1.5 (A4)
- net PI-D0: now also IC1.16 (B3); no longer IC2.11 (B8)
- net PI-D1: now also IC1.17 (B2); no longer IC2.12 (B7)
- net PI-D2: now also IC1.18 (B1); no longer IC2.13 (B6)
- net PI-DP: now also IC1.15 (B4); no longer IC1.18 (B1)
Other:
- note added: "08-Sep-2022"
- note added: "2.6d"
- note removed: "03-Apr-2022"
- note removed: "2.6"
